File: LNA1109.kicad_pcb (KiCad board)
At the start: 4 copper layers, 11.7 x 8.7 mm, 25 parts, among them P1 SMA-KIT-1.5MF, U1 SWITCH, U2 SWITCH, U3 LNA, U4 SAW

Commit message: correct C7 and C8 part selection
Parts:
- C7, C8: value 47pF -> 100pF
Changed lines of the file:
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@@
       (effects (font (size 0.4064 0.4064) (thickness 0.1016)))
     )
-    (fp_text value 47pF (at 0 0.0508 90) (layer F.SilkS) hide
+    (fp_text value 100pF (at 0 0.0508 90) (layer F.SilkS) hide
       (effects (font (size 0.4064 0.4064) (thickness 0.1016)))
     )
@@
       (effects (font (size 0.4064 0.4064) (thickness 0.1016)))
     )
-    (fp_text value 47pF (at 0 0.0508 90) (layer F.SilkS) hide
+    (fp_text value 100pF (at 0 0.0508 90) (layer F.SilkS) hide
       (effects (font (size 0.4064 0.4064) (thickness 0.1016)))
     )
